File: oskar_optocoupler_carrier_pcb.sch (KiCad schematic (older format))
At the start: 5 parts, among them J1 1x3 molex, J2 screw hole, U1 KTIR0611S

Commit message: Assembly and testing time fix for pull-up resistor value.
Parts:
- R2: value 1.5k -> 10k
Changed lines of the file:
@@
 P 3200 1200
 F 0 "R2" H 3141 1154 50  0000 R CNN
-F 1 "1.5k" H 3141 1245 50  0000 R CNN
+F 1 "10k" H 3141 1245 50  0000 R CNN
 F 2 "Resistor_THT:R_Axial_DIN0207_L6.3mm_D2.5mm_P10.16mm_Horizontal" H 3200 1200 50  0001 C CNN
 F 3 "~" H 3200 1200 50  0001 C CNN
